File: controller-pcb/kinesis-80.kicad_sch (KiCad schematic)
At the start: 23 parts, among them J1 Conn_01x07, J2 Conn_01x07, J3 Conn_01x11, J4 Conn_01x11, J5 Conn_01x07, J6 Conn_01x07, J7 Conn_02x04_Odd_Even, J8 Conn_02x04_Odd_Even, U1 weact_STM32F4x1

Commit message: Updated documentation
Other:
- title: Kinesis80 keyboard controller -> kinBP keyboard controller
